File: Hardware/KiCad_Files/Touch_Drum_Built-in_Audio/Touch_Drum_Built-in_Audio.kicad_pcb (KiCad board)
At the start: 2 copper layers, 71.1 x 97.8 mm, 13 parts, among them J1 Conn_01x06, U1 TEENSY_3.2_FULL_PINS, U2 Audio_Shield

Commit message: Updating Millable Version
Parts:
- added H1: STAND-OFF, Hardware:STAND-OFF, F.Cu at (139.7, 57.1)
- added H2: STAND-OFF, Hardware:STAND-OFF, F.Cu at (128.3, 43.2)
- added H3: STAND-OFF, Hardware:STAND-OFF, F.Cu at (139.7, 87.6)
- added H4: STAND-OFF, Hardware:STAND-OFF, F.Cu at (212.1, 43.2)
- added H5: STAND-OFF, Hardware:STAND-OFF, F.Cu at (212.1, 133.3)
- added H6: STAND-OFF, Hardware:STAND-OFF, F.Cu at (128.3, 133.3)
Other:
- board size 71.1 x 97.8 mm -> 91.4 x 97.8 mm
Changed lines of the file:
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@@
   (general
     (thickness 1.6)
-    (drawings 10)
+    (drawings 9)
     (tracks 120)
     (zones 0)
-    (modules 13)
+    (modules 19)
     (nets 24)
   )
@@
     (mod_text_size 1 1)
     (mod_text_width 0.15)
-    (pad_size 12.7 12.7)
-    (pad_drill 0)
+    (pad_size 6.05 6.05)
+    (pad_drill 6.05)
     (pad_to_mask_clearance 0.2)
     (aux_axis_origin 0 0)
@@
       (net 16 TOUCH_9) (solder_mask_margin 0.1016))
   )
+  (module Hardware:STAND-OFF (layer F.Cu)
+    (at 139.7 57.15)
+    (descr "STANDOFF (#4 SCREW)")
+    (tags "STANDOFF (#4 SCREW)")
+    (attr virtual)
+    (fp_text reference H1 (at 0 -3.302) (layer F.SilkS)
+      (effects (font (size 0.6096 0.6096) (thickness 0.127)))
+    )
+    (fp_text value STAND-OFF (at 0 3.429) (layer F.SilkS)
+      (effects (font (size 0.6096 0.6096) (thickness 0.127)))
+    )
+    (fp_arc (start 0 0) (end 0 1.8542) (angle 180) (layer F.SilkS) (width 0.2032))
+    (fp_arc (start 0 0) (end 0 -1.8542) (angle 180) (layer F.SilkS) (width 0.2032))
+    (fp_arc (start 0 0) (end 0 1.8542) (angle 180) (layer F.SilkS) (width 0.2032))
+    (fp_arc (start 0 0) (end 0 -1.8542) (angle 180) (layer F.SilkS) (width 0.2032))
+    (fp_circle (center 0 0) (end 0 -2.794) (layer F.CrtYd) (width 0.127))
+    (pad "" np_thru_hole circle (at 0 0) (size 6.05 6.05) (drill 6.05) (layers *.Cu *.Mask)
+      (solder_mask_margin 0.1016))
+  )
+  (module Hardware:STAND-OFF (layer F.Cu)
+    (at 128.27 43.18)
+    (descr "STANDOFF (#4 SCREW)")
+    (tags "STANDOFF (#4 SCREW)")
+    (attr virtual)
+    (fp_text reference H2 (at 0 -3.302) (layer F.SilkS)
+      (effects (font (size 0.6096 0.6096) (thickness 0.127)))
+    )
+    (fp_text value STAND-OFF (at 0 3.429) (layer F.SilkS)
+      (effects (font (size 0.6096 0.6096) (thickness 0.127)))
+    )
+    (fp_circle (center 0 0) (end 0 -2.794) (layer F.CrtYd) (width 0.127))
+    (fp_arc (start 0 0) (end 0 -1.8542) (angle 180) (layer F.SilkS) (width 0.2032))
+    (fp_arc (start 0 0) (end 0 1.8542) (angle 180) (layer F.SilkS) (width 0.2032))
+    (fp_arc (start 0 0) (end 0 -1.8542) (angle 180) (layer F.SilkS) (width 0.2032))
+    (fp_arc (start 0 0) (end 0 1.8542) (angle 180) (layer F.SilkS) (width 0.2032))
+    (pad "" np_thru_hole circle (at 0 0) (size 3.302 3.302) (drill 3.302) (layers *.Cu *.Mask)
+      (solder_mask_margin 0.1016))
+  )
+  (module Hardware:STAND-OFF (layer F.Cu)
+    (at 139.7 87.63)
+    (descr "STANDOFF (#4 SCREW)")
+    (tags "STANDOFF (#4 SCREW)")
+    (attr virtual)
+    (fp_text reference H3 (at 0 -3.302) (layer F.SilkS)
+      (effects (font (size 0.6096 0.6096) (thickness 0.127)))
+    )
+    (fp_text value STAND-OFF (at 0 3.429) (layer F.SilkS)
+      (effects (font (size 0.6096 0.6096) (thickness 0.127)))
+    )
+    (fp_arc (start 0 0) (end 0 1.8542) (angle 180) (layer F.SilkS) (width 0.2032))
+    (fp_arc (start 0 0) (end 0 -1.8542) (angle 180) (layer F.SilkS) (width 0.2032))
+    (fp_arc (start 0 0) (end 0 1.8542) (angle 180) (layer F.SilkS) (width 0.2032))
+    (fp_arc (start 0 0) (end 0 -1.8542) (angle 180) (layer F.SilkS) (width 0.2032))
+    (fp_circle (center 0 0) (end 0 -2.794) (layer F.CrtYd) (width 0.127))
+    (pad "" np_thru_hole circle (at 0 0) (size 6.05 6.05) (drill 6.05) (layers *.Cu *.Mask)
+      (solder_mask_margin 0.1016))
+  )
+  (module Hardware:STAND-OFF (layer F.Cu)
+    (at 212.09 43.18)
+    (descr "STANDOFF (#4 SCREW)")
+    (tags "STANDOFF (#4 SCREW)")
+    (attr virtual)
+    (fp_text reference H4 (at 0 -3.302) (layer F.SilkS)
+      (effects (font (size 0.6096 0.6096) (thickness 0.127)))
+    )
+    (fp_text value STAND-OFF (at 0 3.429) (layer F.SilkS)
+      (effects (font (size 0.6096 0.6096) (thickness 0.127)))
+    )
+    (fp_circle (center 0 0) (end 0 -2.794) (layer F.CrtYd) (width 0.127))
+    (fp_arc (start 0 0) (end 0 -1.8542) (angle 180) (layer F.SilkS) (width 0.2032))
+    (fp_arc (start 0 0) (end 0 1.8542) (angle 180) (layer F.SilkS) (width 0.2032))
+    (fp_arc (start 0 0) (end 0 -1.8542) (angle 180) (layer F.SilkS) (width 0.2032))
+    (fp_arc (start 0 0) (end 0 1.8542) (angle 180) (layer F.SilkS) (width 0.2032))
+    (pad "" np_thru_hole circle (at 0 0) (size 3.302 3.302) (drill 3.302) (layers *.Cu *.Mask)
+      (solder_mask_margin 0.1016))
+  )
+  (module Hardware:STAND-OFF (layer F.Cu)
+    (at 212.09 133.35)
+    (descr "STANDOFF (#4 SCREW)")
+    (tags "STANDOFF (#4 SCREW)")
+    (attr virtual)
+    (fp_text reference H5 (at 0 -3.302) (layer F.SilkS)
+      (effects (font (size 0.6096 0.6096) (thickness 0.127)))
+    )
+    (fp_text value STAND-OFF (at 0 3.429) (layer F.SilkS)
+      (effects (font (size 0.6096 0.6096) (thickness 0.127)))
+    )
+    (fp_arc (start 0 0) (end 0 1.8542) (angle 180) (layer F.SilkS) (width 0.2032))
+    (fp_arc (start 0 0) (end 0 -1.8542) (angle 180) (layer F.SilkS) (width 0.2032))
+    (fp_arc (start 0 0) (end 0 1.8542) (angle 180) (layer F.SilkS) (width 0.2032))
+    (fp_arc (start 0 0) (end 0 -1.8542) (angle 180) (layer F.SilkS) (width 0.2032))
+    (fp_circle (center 0 0) (end 0 -2.794) (layer F.CrtYd) (width 0.127))
+    (pad "" np_thru_hole circle (at 0 0) (size 3.302 3.302) (drill 3.302) (layers *.Cu *.Mask)
+      (solder_mask_margin 0.1016))
+  )
+  (module Hardware:STAND-OFF (layer F.Cu)
+    (at 128.27 133.35)
+    (descr "STANDOFF (#4 SCREW)")
+    (tags "STANDOFF (#4 SCREW)")
+    (attr virtual)
+    (fp_text reference H6 (at 0 -3.302) (layer F.SilkS)
+      (effects (font (size 0.6096 0.6096) (thickness 0.127)))
+    )
+    (fp_text value STAND-OFF (at 0 3.429) (layer F.SilkS)
+      (effects (font (size 0.6096 0.6096) (thickness 0.127)))
+    )
+    (fp_circle (center 0 0) (end 0 -2.794) (layer F.CrtYd) (width 0.127))
+    (fp_arc (start 0 0) (end 0 -1.8542) (angle 180) (layer F.SilkS) (width 0.2032))
+    (fp_arc (start 0 0) (end 0 1.8542) (angle 180) (layer F.SilkS) (width 0.2032))
+    (fp_arc (start 0 0) (end 0 -1.8542) (angle 180) (layer F.SilkS) (width 0.2032))
+    (fp_arc (start 0 0) (end 0 1.8542) (angle 180) (layer F.SilkS) (width 0.2032))
+    (pad "" np_thru_hole circle (at 0 0) (size 3.302 3.302) (drill 3.302) (layers *.Cu *.Mask)
+      (solder_mask_margin 0.1016))
+  )
   (dimension 97.79 (width 0.3) (layer B.SilkS)
     (gr_text "3.8500 in" (at 226.89 88.265 270) (layer B.SilkS)
@@
     (arrow2b (pts (xy 224.79 39.37) (xy 225.376421 40.496504)))
   )
-  (dimension 69.85 (width 0.3) (layer B.SilkS)
-    (gr_text "2.7500 in" (at 180.975 143.07) (layer B.SilkS)
-      (effects (font (size 1.5 1.5) (thickness 0.3)))
-    )
-    (feature1 (pts (xy 215.9 137.16) (xy 215.9 141.556421)))
-    (feature2 (pts (xy 146.05 137.16) (xy 146.05 141.556421)))
-    (crossbar (pts (xy 146.05 140.97) (xy 215.9 140.97)))
-    (arrow1a (pts (xy 215.9 140.97) (xy 214.773496 141.556421)))
-    (arrow1b (pts (xy 215.9 140.97) (xy 214.773496 140.383579)))
-    (arrow2a (pts (xy 146.05 140.97) (xy 147.176504 141.556421)))
-    (arrow2b (pts (xy 146.05 140.97) (xy 147.176504 140.383579)))
-  )
-  (gr_line (start 156.21 39.37) (end 144.78 39.37) (layer Edge.Cuts) (width 0.2))
-  (gr_line (start 144.78 45.72) (end 144.78 39.37) (layer Edge.Cuts) (width 0.2))
-  (gr_line (start 144.78 114.3) (end 144.78 45.72) (layer Edge.Cuts) (width 0.2))
+  (gr_line (start 156.21 39.37) (end 124.46 39.37) (layer Edge.Cuts) (width 0.2))
+  (gr_line (start 124.46 45.72) (end 124.46 39.37) (layer Edge.Cuts) (width 0.2))
+  (gr_line (start 124.46 114.3) (end 124.46 45.72) (layer Edge.Cuts) (width 0.2))
   (gr_line (start 215.9 39.37) (end 156.21 39.37) (layer Edge.Cuts) (width 0.2))
   (gr_line (start 215.9 66.04) (end 215.9 39.37) (layer Edge.Cuts) (width 0.2))
   (gr_line (start 215.9 137.16) (end 215.9 66.04) (layer Edge.Cuts) (width 0.2))
-  (gr_line (start 144.78 137.16) (end 215.9 137.16) (layer Edge.Cuts) (width 0.2))
-  (gr_line (start 144.78 114.3) (end 144.78 137.16) (layer Edge.Cuts) (width 0.2))
+  (gr_line (start 124.46 137.16) (end 215.9 137.16) (layer Edge.Cuts) (width 0.2))
+  (gr_line (start 124.46 114.3) (end 124.46 137.16) (layer Edge.Cuts) (width 0.2))
   (segment (start 189.23 68.58) (end 191.77 66.04) (width 0.406) (layer B.Cu) (net 1))
   (segment (start 191.77 66.04) (end 201.93 66.04) (width 0.406) (layer B.Cu) (net 1))
@@
     (polygon
       (pts
-        (xy 144.78 39.37) (xy 215.9 39.37) (xy 215.9 137.16) (xy 144.78 137.16)
+        (xy 124.46 39.37) (xy 195.58 39.37) (xy 195.58 137.16) (xy 124.46 137.16)
       )
     )
