File: Hardware/KiCad_Files/Touch_Drum_V1/Base/Touch_Drum_V1.kicad_pcb (KiCad board)
At the start: 2 copper layers, 0 parts

Commit message: Mostly complete Top layer PCB of V1 Touch Drum
Other:
- board outline added: 133.4 x 133.3 mm
Changed lines of the file:
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@@
   (general
     (thickness 1.6)
-    (drawings 0)
+    (drawings 1)
     (tracks 0)
     (zones 0)
@@
     (uvia_drill 0.1)
   )
+  (gr_circle (center 107.315 101.6) (end 40.64 101.6) (layer Edge.Cuts) (width 0.15))
 )

Commit message: Adding more reference files
Parts:
- added J1: Conn_01x10, Connectors:1X10_SMD_MALE, B.Cu at (120.7, 121.9)
- added J2: Conn_01x10, Connectors:1X10_SMD_MALE, B.Cu at (97.8, 81.3)
- added JP1: JP_3_1-NC, Jumpers:SMT-JUMPER_3_1-NC_TRACE_SILK, B.Cu at (-99.3, 61.0)
- added JP2: JP_3_1-NC, Jumpers:SMT-JUMPER_3_1-NC_TRACE_SILK, B.Cu at (-93.5, 61.0)
- added JP3: JP_3_1-NC, Jumpers:SMT-JUMPER_3_1-NC_TRACE_SILK, B.Cu at (-62.2, 61.0)
- added JP4: JP_3_1-NC, Jumpers:SMT-JUMPER_3_1-NC_TRACE_SILK, B.Cu at (-56.1, 61.0)
- added L1: LOGO, Openponics_Logos:TouchDrumLogo, F.Cu at (-77.5, 119.4)
- added TP1: PAD_0, Openponics_Hardware:PAD.LARGE_0.5INCH, F.Cu at (-92.7, 111.8)
- added TP10: PAD_9, Openponics_Hardware:PAD.LARGE_0.5INCH, F.Cu at (-62.2, 111.8)
- added TP2: PAD_1, Openponics_Hardware:PAD.LARGE_1.0INCH, F.Cu at (-115.6, 134.6)
- added TP3: PAD_2, Openponics_Hardware:PAD.LARGE_1.25INCH, F.Cu at (-77.5, 142.2)
- added TP4: PAD_3, Openponics_Hardware:PAD.LARGE_1.0INCH, F.Cu at (-40.6, 134.6)
- added TP5: PAD_4, Openponics_Hardware:PAD.LARGE_1.25INCH, F.Cu at (-33.0, 97.8)
- added TP6: PAD_5, Openponics_Hardware:PAD.LARGE_1.25INCH, F.Cu at (-77.5, 52.1)
- added TP7: PAD_6, Openponics_Hardware:PAD.LARGE_1.0INCH, F.Cu at (-115.6, 61.0)
- added TP8: PAD_7, Openponics_Hardware:PAD.LARGE_1.25INCH, F.Cu at (-123.2, 97.8)
- added TP9: PAD_8, Openponics_Hardware:PAD.LARGE_1.0INCH, F.Cu at (-40.6, 61.0)
- added U1: TeensyView, Openponics_Templates:TeensyView, F.Cu at (-94.0, 106.7)
- added VR1: TRIMPOT, Openponics_Templates:Panel_Mount_Potentiometer, B.Cu at (-96.5, 78.7)
- added VR2: TRIMPOT, Openponics_Templates:Panel_Mount_Potentiometer, B.Cu at (-58.9, 78.7)
Routing:
- net (no net): track 0.00 -> 719.5 mm, vias 0 -> 14
- added copper zone on B.Cu, net (none)
Other:
- board size 133.4 x 133.3 mm -> 266.8 x 133.3 mm
- board text added: "3.3V"
- board text added: "GND"
- board text added: "KEY"
- board text added: "SCALE"
